Commit message: added the models of the boxes , added simple servoing algorithm and yet to add a circle on the aruco detections

File: urdf/mogi_bot.urdf (robot description, URDF)
Before this commit: robot mogi_bot, 9 links, 8 joints
Links:
- link base_link: geometry collision box size=.4 .2 .1; collision sphere radius=0.0499
- link left_wheel: geometry collision cylinder length=.05 radius=.1; visual mesh filename=package://assign1/meshes/wheel.dae
- link right_wheel: geometry collision cylinder length=.05 radius=.1; visual mesh filename=package://assign1/meshes/wheel.dae
- link scan_link: geometry collision box size=.1 .1 .1; visual mesh filename=package://assign1/meshes/lidar.dae
